Commit message: Add Depth Camera

File: mo2bot_description/urdf/mo2bot.xacro (robot description, xacro)
@@ -406,5 +406,5 @@
               <cylinder radius="0.0525" length="0.03"/>
             </geometry>
-            <material name="black"/>
+            <material name="grey"/>
           </visual>
           <!--Body-->
@@ -450,4 +450,40 @@
           <child link="camera"/>
         </joint>
+        <!-- Depth Camera, Back -->
+        <!-- ZED Cam https://www.stereolabs.com/zed/ -->
+        <link name="dcam_back">
+          <collision>
+            <origin xyz="0 0 0" rpy="0 0 0"/>
+            <geometry>
+              <box size=".03 .175 .033"/>
+            </geometry>
+          </collision>
+          <visual>
+            <origin xyz="0 0 0" rpy="0 0 0"/>
+            <geometry>
+              <box size=".03 .175 .033"/>
+            </geometry>
+            <material name="grey"/>
+          </visual>
+          <inertial>
+            <mass value="${cameraMass}" />
+            <origin xyz="0 0 0" rpy="0 0 0"/>
+            <box_inertia m="0.159" x=".03" y=".175" z=".033" />
+            <inertia ixx="1e-6" ixy="0" ixz="0" iyy="1e-6" iyz="0" izz="1e-6" />
+          </inertial>
+        </link>
+        <joint name="joint_dcam_back" type="fixed">
+          <axis xyz="0 1 0" />
+          <origin xyz="-.27 0 0.2" rpy="0 0 3.1416"/>
+          <parent link="chassis"/>
+          <child link="dcam_back"/>
+        </joint>
+        <!--Camera to Depth link -->
+        <joint name="joint_dcam_back_depth" type="fixed">
+    <origin xyz="0 0 0" rpy="${-3.1416/2} 0 ${-3.1416/2} "/>
+    <parent link="dcam_back"/>
+    <child link="dcam_back_depth"/>
+  </joint>
+  <link name="dcam_back_depth"></link>
         <!-- Hokuyo Laser -->
         <!--joint name="hokuyo_joint" type="fixed">

Commit message: Add IMU

File: mo2bot_description/urdf/mo2bot.xacro (robot description, xacro)
@@ -446,5 +446,5 @@
         <joint name="camera_joint" type="fixed">
           <axis xyz="0 1 0" />
-          <origin xyz=".2 0 0" rpy="0 0 0"/>
+          <origin xyz="-.27 0 0.2" rpy="0 0 0"/>
           <parent link="chassis"/>
           <child link="camera"/>
@@ -475,5 +475,5 @@
         <joint name="joint_dcam_back" type="fixed">
           <axis xyz="0 1 0" />
-          <origin xyz="-.27 0 0.2" rpy="0 0 3.1416"/>
+          <origin xyz=".27 0 0.32" rpy="0 0 0"/>
           <parent link="chassis"/>
           <child link="dcam_back"/>
@@ -486,29 +486,61 @@
   </joint>
   <link name="dcam_back_depth"></link>
-        <!-- Hokuyo Laser -->
-        <!--joint name="hokuyo_joint" type="fixed">
-        <axis xyz="0 1 0" />
-        <origin xyz=".15 0 .1" rpy="0 0 0"/>
-        <parent link="chassis"/>
-        <child link="hokuyo"/>
-      </joint>
-      <link name="hokuyo">
-      <collision>
+  <!-- IMU -->
+  <!-- With breadboard -->
+  <link name="imu_link">
+    <collision>
       <origin xyz="0 0 0" rpy="0 0 0"/>
       <geometry>
-      <box size="0.1 0.1 0.1"/>
-    </geometry>
-  </collision>
-  <visual>
-  <origin xyz="0 0 0" rpy="0 0 0"/>
-  <geometry>
-  <mesh filename="package://mo2bot_description/meshes/hokuyo.dae"/>
-</geometry>
-</visual>
-<inertial>
-<mass value="1e-5" />
-<origin xyz="0 0 0" rpy="0 0 0"/>
-<inertia ixx="1e-6" ixy="0" ixz="0" iyy="1e-6" iyz="0" izz="1e-6" />
-</inertial>
-</link-->
+        <box size=".0168 .0212 .005"/>
+      </geometry>
+    </collision>
+    <visual>
+      <origin xyz="0 0 0" rpy="0 0 0"/>
+      <geometry>
+        <box size=".0168 .0212 .005"/>
+      </geometry>
+      <material name="grey"/>
+    </visual>
+    <inertial>
+      <mass value="0.01" />
+      <origin xyz="0 0 0" rpy="0 0 0"/>
+      <box_inertia m="0.01" x=".0168" y=".0212" z=".005" />
+      <inertia ixx="1e-6" ixy="0" ixz="0" iyy="1e-6" iyz="0" izz="1e-6" />
+    </inertial>
+  </link>
+  <joint name="joint_imu" type="fixed">
+    <axis xyz="0 1 0" />
+    <origin xyz="0.1 0.1 0.1" rpy="0 0 1.57"/>
+    <parent link="chassis"/>
+    <child link="imu_link"/>
+  </joint>
+  <!-- LCD Display -->
+  <!--  -->
+  <link name="lcd_screen">
+    <collision>
+      <origin xyz="0 0 0" rpy="0 0 0"/>
+      <geometry>
+        <box size=".150 .255 .005"/>
+      </geometry>
+    </collision>
+    <visual>
+      <origin xyz="0 0 0" rpy="0 0 0"/>
+      <geometry>
+        <box size=".150 .255 .005"/>
+      </geometry>
+      <material name="grey"/>
+    </visual>
+    <inertial>
+      <mass value="${cameraMass}" />
+      <origin xyz="0 0 0" rpy="0 0 0"/>
+      <box_inertia m="0.159" x=".150" y=".255" z=".005" />
+      <inertia ixx="1e-6" ixy="0" ixz="0" iyy="1e-6" iyz="0" izz="1e-6" />
+    </inertial>
+  </link>
+  <joint name="joint_lcd_screen" type="fixed">
+    <axis xyz="0 1 0" />
+    <origin xyz=".26 0 0.13" rpy="0 1.57 0"/>
+    <parent link="chassis"/>
+    <child link="lcd_screen"/>
+  </joint>
 </robot>

Commit message: Cleanup code

File: mo2bot_description/urdf/mo2bot.xacro (robot description, xacro)
@@ -1,6 +1,14 @@
 <?xml version='1.0'?>
-<robot name="myrobot" xmlns:xacro="http://www.ros.org/wiki/xacro">
+<robot name="momobot" xmlns:xacro="http://www.ros.org/wiki/xacro">
+  <!-- Params -->
   <xacro:property name="cameraSize" value="0.05"/>
   <xacro:property name="cameraMass" value="0.1"/>
+  <!-- Trolley wheels -->
+  <xacro:property name="wheel_t_radius" value="0.05"/>
+  <xacro:property name="wheel_t_length" value="0.03"/>
+  <!-- Main (Scooter) wheels -->
+  <xacro:property name="wheel_m_radius" value="0.1"/>
+  <xacro:property name="wheel_m_length" value="0.05"/>
+  <!-- Dependencies -->
   <xacro:include filename="$(find mo2bot_description)/urdf/mo2bot.gazebo" />
   <xacro:include filename="$(find mo2bot_description)/urdf/materials.xacro" />
@@ -52,86 +60,10 @@
       </visual>
     </link>
-    <!--Caster Wheels-->
-    <!--link name='caster_left'>
-      <collision name='caster_collision_left'>
-        <origin xyz="0 0 0" rpy=" 0 0 0"/>
-        <geometry>
-          <sphere radius="0.05"/>
-        </geometry>
-        <surface>
-          <friction>
-            <ode>
-              <mu>0</mu>
-              <mu2>0</mu2>
-              <slip1>1.0</slip1>
-              <slip2>1.0</slip2>
-            </ode>
-          </friction>
-        </surface>
-      </collision>
-      <visual name='caster_visual_left'>
-        <origin xyz="0 0 0" rpy=" 0 0 0"/>
-        <geometry>
-          <sphere radius="0.05"/>
-        </geometry>
-        <material name="grey"/>
-      </visual>
-      <inertial>
-        <mass value="1"/>
-        <origin rpy="0 0 0" xyz="0 0 0"/>
-        <inertia ixx="0.0027" iyy="0.0027" izz="0.005" ixy="0" ixz="0" iyz="0"/>
-      </inertial>
-    </link-->
-    <!-- Caster joint, Left -->
-    <!--joint name="cst_joint_left" type="continuous">
-      <axis xyz="1 1 0"/>
-      <parent link="chassis"/>
-      <child link="caster_left"/>
-      <origin xyz="0.22 -0.24 -0.4" rpy="0 0 0" />
-    </joint-->
-    <!--Caster wheel, Right-->
-    <!--link name='caster_right'>
-      <collision name='caster_collision_right'>
-        <origin xyz="0 0 0" rpy=" 0 0 0"/>
-        <geometry>
-          <sphere radius="0.05"/>
-        </geometry>
-        <surface>
-          <friction>
-            <ode>
-              <mu>0</mu>
-              <mu2>0</mu2>
-              <slip1>1.0</slip1>
-              <slip2>1.0</slip2>
-            </ode>
-          </friction>
-        </surface>
-      </collision>
-      <visual name='caster_visual_right'>
-        <origin xyz="0 0 0" rpy=" 0 0 0"/>
-        <geometry>
-          <sphere radius="0.05"/>
-        </geometry>
-        <material name="grey"/>
-      </visual>
-      <inertial>
-        <mass value="1"/>
-        <origin rpy="0 0 0" xyz="0 0 0"/>
-        <inertia ixx="0.0027" iyy="0.0027" izz="0.005" ixy="0" ixz="0" iyz="0"/>
-      </inertial>
-    </link-->
-    <!-- Caster joint, right -->
-    <!--joint name="cst_joint_right" type="continuous">
-      <axis xyz="1 1 0"/>
-      <parent link="chassis"/>
-      <child link="caster_right"/>
-      <origin xyz="0.22 0.24 -0.4" rpy="0 0 0"/>
-    </joint-->
-<!--Left trolley wheel-->
+    <!--Left trolley wheel-->
     <link name='trolleyW_wheel_front_left'>
       <collision name='collision_trolleyW_wheel_front_left'>
         <origin xyz="0 0 0" rpy=" 0 1.5707 1.5707"/>
         <geometry>
-          <cylinder radius="0.05" length="0.03"/>
+          <cylinder radius="${wheel_t_radius}" length="${wheel_t_length}"/>
         </geometry>
         <surface>
@@ -149,5 +81,5 @@
         <origin xyz="0 0 0" rpy=" 0 1.5707 1.5707"/>
         <geometry>
-          <cylinder radius="0.05" length="0.03"/>
+          <cylinder radius="${wheel_t_radius}" length="${wheel_t_length}"/>
         </geometry>
         <material name="grey"/>
@@ -161,66 +93,66 @@
           iyy="560e-6" iyz="0"
           izz="0.001"   />
-      </inertial>
-    </link>
-    <joint name="joint_trolleyW_wheel_front_left" type="continuous">
-      <axis xyz="0 1 0"/>
-      <parent link="trolleyW_holder_front_left"/>
-      <child link="trolleyW_wheel_front_left"/>
-      <origin xyz="-0.04 0 -0.06" rpy="0 0 0" />
-    </joint>
-<!--Trolley wheel holder attachment-->
-    <link name='trolleyW_holder_front_left'>
-      <collision name='collision_trolleyW_holder_front_left'>
-        <origin xyz="-0.03 0 -0.0075" rpy=" 0 0 0"/>
-        <geometry>
-          <box size=".1 .03 .015"/>
-        </geometry>
-        <surface>
-          <friction>
-            <ode>
-              <mu>0</mu>
-              <mu2>0</mu2>
-              <slip1>1.0</slip1>
-              <slip2>1.0</slip2>
-            </ode>
-          </friction>
-        </surface>
-      </collision>
-      <visual name='visual_trolleyW_holderHorizontal_front_left'>
-        <origin xyz="-0.03 0 -0.0075" rpy=" 0 0 0"/>
-        <geometry>
-          <box size=".1 .03 .015"/>
-        </geometry>
-        <material name="grey"/>
-      </visual>
-      <visual name='visual_trolleyW_holderVertical_front_left'>
-        <origin xyz="-0.04 0 -0.03" rpy=" 0 0 0"/>
-        <geometry>
-          <box size=".015 .03 .06"/>
-        </geometry>
-        <material name="grey"/>
-      </visual>
-      <!-- Inertia calculation based on m=0.05, w = 0.1, h=0.03, d=0.015-->
-      <inertial>
-        <mass value="1"/>
-        <origin rpy="-0.02 0 0" xyz="0 0 0"/>
-        <inertia
-          ixx="4.6875e-6" ixy="0" ixz="0"
-          iyy="42.6041e-6" iyz="0"
-          izz="45.4167e-6"   />
-      </inertial>
-    </link>
-    <joint name="joint_trolleyW_front_left" type="continuous">
-      <axis xyz="0 0 1"/>
-      <parent link="base_link"/>
-      <child link="trolleyW_holder_front_left"/>
-      <origin xyz="0.22 0.22 -0.345" rpy="0 0 0" />
-    </joint>
-    <!--Right trolley wheel-->
+        </inertial>
+      </link>
+      <joint name="joint_trolleyW_wheel_front_left" type="continuous">
+        <axis xyz="0 1 0"/>
+        <parent link="trolleyW_holder_front_left"/>
+        <child link="trolleyW_wheel_front_left"/>
+        <origin xyz="-0.04 0 -0.06" rpy="0 0 0" />
+      </joint>
+      <!--Trolley wheel holder attachment-->
+      <link name='trolleyW_holder_front_left'>
+        <collision name='collision_trolleyW_holder_front_left'>
+          <origin xyz="-0.03 0 -0.0075" rpy=" 0 0 0"/>
+          <geometry>
+            <box size=".1 .03 .015"/>
+          </geometry>
+          <surface>
+            <friction>
+              <ode>
+                <mu>0</mu>
+                <mu2>0</mu2>
+                <slip1>1.0</slip1>
+                <slip2>1.0</slip2>
+              </ode>
+            </friction>
+          </surface>
+        </collision>
+        <visual name='visual_trolleyW_holderHorizontal_front_left'>
+          <origin xyz="-0.03 0 -0.0075" rpy=" 0 0 0"/>
+          <geometry>
+            <box size=".1 .03 .015"/>
+          </geometry>
+          <material name="grey"/>
+        </visual>
+        <visual name='visual_trolleyW_holderVertical_front_left'>
+          <origin xyz="-0.04 0 -0.03" rpy=" 0 0 0"/>
+          <geometry>
+            <box size=".015 .03 .06"/>
+          </geometry>
+          <material name="grey"/>
+        </visual>
+        <!-- Inertia calculation based on m=0.05, w = 0.1, h=0.03, d=0.015-->
+        <inertial>
+          <mass value="1"/>
+          <origin rpy="-0.02 0 0" xyz="0 0 0"/>
+          <inertia
+            ixx="4.6875e-6" ixy="0" ixz="0"
+            iyy="42.6041e-6" iyz="0"
+            izz="45.4167e-6"   />
+          </inertial>
+        </link>
+        <joint name="joint_trolleyW_front_left" type="continuous">
+          <axis xyz="0 0 1"/>
+          <parent link="base_link"/>
+          <child link="trolleyW_holder_front_left"/>
+          <origin xyz="0.22 0.22 -0.345" rpy="0 0 0" />
+        </joint>
+        <!--Right trolley wheel-->
         <link name='trolleyW_wheel_front_right'>
           <collision name='collision_trolleyW_wheel_front_right'>
             <origin xyz="0 0 0" rpy=" 0 1.5707 1.5707"/>
             <geometry>
-              <cylinder radius="0.05" length="0.03"/>
+              <cylinder radius="${wheel_t_radius}" length="${wheel_t_length}"/>
             </geometry>
             <surface>
@@ -238,5 +170,5 @@
             <origin xyz="0 0 0" rpy=" 0 1.5707 1.5707"/>
             <geometry>
-              <cylinder radius="0.05" length="0.03"/>
+              <cylinder radius="${wheel_t_radius}" length="${wheel_t_length}"/>
             </geometry>
             <material name="grey"/>
@@ -250,288 +182,291 @@
               iyy="560e-6" iyz="0"
               izz="0.001"   />
-          </inertial>
-        </link>
-        <joint name="joint_trolleyW_wheel_front_right" type="continuous">
-          <axis xyz="0 1 0"/>
-          <parent link="trolleyW_holder_front_right"/>
-          <child link="trolleyW_wheel_front_right"/>
-          <origin xyz="-0.04 0 -0.06" rpy="0 0 0" />
-        </joint>
-    <!--Trolley wheel holder attachment-->
-        <link name='trolleyW_holder_front_right'>
-          <collision name='collision_trolleyW_holder_front_right'>
-            <origin xyz="-0.03 0 -0.0075" rpy=" 0 0 0"/>
-            <geometry>
-              <box size=".1 .03 .015"/>
-            </geometry>
-            <surface>
-              <friction>
-                <ode>
-                  <mu>0</mu>
-                  <mu2>0</mu2>
-                  <slip1>1.0</slip1>
-                  <slip2>1.0</slip2>
-                </ode>
-              </friction>
-            </surface>
-          </collision>
-          <visual name='visual_trolleyW_holderHorizontal_front_right'>
-            <origin xyz="-0.03 0 -0.0075" rpy=" 0 0 0"/>
-            <geometry>
-              <box size=".1 .03 .015"/>
-            </geometry>
-            <material name="grey"/>
-          </visual>
-          <visual name='visual_trolleyW_holderVertical_front_right'>
-            <origin xyz="-0.04 0 -0.03" rpy=" 0 0 0"/>
-            <geometry>
-              <box size=".015 .03 .06"/>
-            </geometry>
-            <material name="grey"/>
-          </visual>
-          <!-- Inertia calculation based on m=0.05, w = 0.1, h=0.03, d=0.015-->
-          <inertial>
-            <mass value="1"/>
-            <origin rpy="-0.02 0 0" xyz="0 0 0"/>
-            <inertia
-              ixx="4.6875e-6" ixy="0" ixz="0"
-              iyy="42.6041e-6" iyz="0"
-              izz="45.4167e-6"   />
-          </inertial>
-        </link>
-        <joint name="joint_trolleyW_front_right" type="continuous">
-          <axis xyz="0 0 1"/>
-          <parent link="base_link"/>
-          <child link="trolleyW_holder_front_right"/>
-          <origin xyz="0.22 -0.22 -0.345" rpy="0 0 0" />
-        </joint>
-    <!--Main Wheels-->
-    <!-- Inertia calculation based on m=2, h=0.05, r=0.1-->
-    <link name="left_wheel">
-      <!--origin xyz="0.1 0.13 0.1" rpy="0 1.5707 1.5707"/-->
-      <collision name="collision">
-        <origin xyz="0 0 0" rpy="0 1.5707 1.5707"/>
-        <geometry>
-          <cylinder radius="0.1" length="0.05"/>
-        </geometry>
-      </collision>
-      <visual name="left_wheel_visual">
-        <origin xyz="0 0 0" rpy="0 1.5707 1.5707"/>
-        <geometry>
-          <cylinder radius="0.1" length="0.05"/>
-        </geometry>
-        <material name="black"/>
-      </visual>
-      <inertial>
-        <origin xyz="0 0 0" rpy="0 1.5707 1.5707"/>
-        <mass value="5"/>
-        <inertia
-          ixx="5.4167e-3" ixy="0.0" ixz="0.0"
-          iyy="5.4167e-3" iyz="0.0"
-          izz="0.01"/>
-        </inertial>
-      </link>
-      <!--Left wheel joint-->
-      <joint type="continuous" name="left_wheel_joint">
-        <origin xyz="-0.124 0.19 -.35" rpy="0 0 0"/>
-        <!--origin xyz="0.1 0.13 0" rpy="0 1.5707 1.5707"/-->
-        <child link="left_wheel"/>
-        <parent link="base_link"/>
-        <axis xyz="0 1 0" rpy="0 0 0"/>
-        <limit effort="10000" velocity="1000"/>
-        <joint_properties damping="1.0" friction="1.0"/>
-      </joint>
-      <link name="right_wheel">
-        <!--origin xyz="0.1 -0.13 0.1" rpy="0 1.5707 1.5707"/-->
-        <collision name="collision">
-          <origin xyz="0 0 0" rpy="0 1.5707 1.5707"/>
-          <geometry>
-            <cylinder radius="0.1" length="0.05"/>
-          </geometry>
-        </collision>
-        <visual name="right_wheel_visual">
-          <origin xyz="0 0 0" rpy="0 1.5707 1.5707"/>
-          <geometry>
-            <cylinder radius="0.1" length="0.05"/>
-          </geometry>
-          <material name="black"/>
-        </visual>
-        <inertial>
-          <origin xyz="0 0 0" rpy="0 1.5707 1.5707"/>
-          <mass value="5"/>
-          <inertia
-            ixx="5.4167e-3" ixy="0.0" ixz="0.0"
-            iyy="5.4167e-3" iyz="0.0"
-            izz="0.01"/>
-          </inertial>
-        </link>
-        <!--Right Wheel Joint-->
-        <joint type="continuous" name="right_wheel_joint">
-          <origin xyz="-0.124 -0.19 -.35" rpy="0 0 0"/>
-          <!--origin xyz="0.1 -0.13 0" rpy="0 1.5707 1.5707"/-->
-          <child link="right_wheel"/>
-          <parent link="base_link"/>
-          <axis xyz="0 1 0" rpy="0 0 0"/>
-          <limit effort="10000" velocity="1000"/>
-          <joint_properties damping="1.0" friction="1.0"/>
-        </joint>
-        <!--Lidar-->
-        <joint name="sick_joint" type="fixed">
-          <axis xyz="0 1 0" />
-          <origin xyz=".3 0 -.22" rpy="3.1416 0 0"/>
-          <parent link="base_link"/>
-          <child link="sick_l"/>
-        </joint>
-        <!-- SICK Laser -->
-        <link name="sick_l">
-          <collision>
-            <origin xyz="0 0 -0.05" rpy="0 0 0"/>
-            <geometry>
-              <box size="0.105 0.102 0.28"/>
-            </geometry>
-          </collision>
-          <!--Top-->
-          <visual name='sick_visual_top'>
-            <origin xyz="0 0 0" rpy="0 0 0"/>
-            <geometry>
-              <cylinder radius="0.0525" length="0.03"/>
-            </geometry>
-            <material name="grey"/>
-          </visual>
-          <!--Body-->
-          <visual name='sick_visual_body'>
-            <origin xyz="0 0 -0.067" rpy="0 0 0"/>
-            <geometry>
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
Commit message: Shift back camera lower

File: mo2bot_description/urdf/mo2bot.xacro (robot description, xacro)
@@ -349,10 +349,10 @@
                 </inertial>
               </link>
-              <!--Camera-->
-              <link name="camera">
+              <!--Camera, Bottom back-->
+              <link name="cam_back_btm">
                 <collision>
                   <origin xyz="0 0 0" rpy="0 0 0"/>
                   <geometry>
-                    <box size="${cameraSize} ${cameraSize} ${cameraSize}"/>
+                    <box size=".03 .130 .033"/>
                   </geometry>
                 </collision>
@@ -360,12 +360,12 @@
                   <origin xyz="0 0 0" rpy="0 0 0"/>
                   <geometry>
-                    <box size="${cameraSize} ${cameraSize} ${cameraSize}"/>
-                  </geometry>
-                  <material name="green"/>
+                    <box size=".03 .130 .033"/>
+                  </geometry>
+                  <material name="black"/>
                 </visual>
                 <inertial>
                   <mass value="${cameraMass}" />
                   <origin xyz="0 0 0" rpy="0 0 0"/>
-                  <box_inertia m="${cameraMass}" x="${cameraSize}" y="${cameraSize}" z="${cameraSize}" />
+                  <box_inertia m="${cameraMass}" x="0.03" y="0.130" z="0.033" />
                   <inertia ixx="1e-6" ixy="0" ixz="0" iyy="1e-6" iyz="0" izz="1e-6" />
                 </inertial>
@@ -373,7 +373,7 @@
               <joint name="camera_joint" type="fixed">
                 <axis xyz="0 1 0" />
-                <origin xyz="-.27 0 0.2" rpy="0 0 0"/>
-                <parent link="base_link"/>
-                <child link="camera"/>
+                <origin xyz="-.27 0 -0.1" rpy="0 0 3.142"/>
+                <parent link="base_link"/>
+                <child link="cam_back_btm"/>
               </joint>
               <!-- Depth Camera, Back -->
