Commit message: Change camera type
- Change camera from depth camera to stereo camera
- Fix LCD display

File: mo2bot_description/urdf/mo2bot.xacro (robot description, xacro)
@@ -377,7 +377,7 @@
                 <child link="cam_back_btm"/>
               </joint>
-              <!-- Depth Camera, Back -->
+              <!-- Depth Camera, Front -->
               <!-- ZED Cam https://www.stereolabs.com/zed/ -->
-              <link name="dcam_back">
+              <link name="dcam_front">
                 <collision>
                   <origin xyz="0 0 0" rpy="0 0 0"/>
@@ -394,5 +394,5 @@
                 </visual>
                 <inertial>
-                  <mass value="${cameraMass}" />
+                  <mass value="0.159" />
                   <origin xyz="0 0 0" rpy="0 0 0"/>
                   <box_inertia m="0.159" x=".03" y=".175" z=".033" />
@@ -400,17 +400,17 @@
                 </inertial>
               </link>
-              <joint name="joint_dcam_back" type="fixed">
+              <joint name="joint_dcam_front" type="fixed">
                 <axis xyz="0 1 0" />
                 <origin xyz=".27 0 0.32" rpy="0 0 0"/>
                 <parent link="base_link"/>
-                <child link="dcam_back"/>
+                <child link="dcam_front"/>
               </joint>
               <!--Camera to Depth link -->
-              <joint name="joint_dcam_back_depth" type="fixed">
+              <joint name="joint_dcam_front_depth" type="fixed">
                 <origin xyz="0 0 0" rpy="${-3.1416/2} 0 ${-3.1416/2} "/>
-                <parent link="dcam_back"/>
-                <child link="dcam_back_depth"/>
-              </joint>
-              <link name="dcam_back_depth"></link>
+                <parent link="dcam_front"/>
+                <child link="dcam_front_depth"/>
+              </joint>
+              <link name="dcam_front_depth"></link>
               <!-- IMU -->
               <!-- With breadboard -->
@@ -447,5 +447,5 @@
                   <origin xyz="0 0 0" rpy="0 0 0"/>
                   <geometry>
-                    <box size=".150 .255 .005"/>
+                    <box size=".255 .150 .005"/>
                   </geometry>
                 </collision>
@@ -453,5 +453,5 @@
                   <origin xyz="0 0 0" rpy="0 0 0"/>
                   <geometry>
-                    <box size=".150 .255 .005"/>
+                    <box size=".255 .150 .005"/>
                   </geometry>
                   <material name="grey"/>
@@ -460,5 +460,5 @@
                   <mass value="0.2" />
                   <origin xyz="0 0 0" rpy="0 0 0"/>
-                  <box_inertia m="0.159" x=".150" y=".255" z=".005" />
+                  <box_inertia m="0.159" x=".255" y=".150" z=".005" />
                   <inertia ixx="1e-6" ixy="0" ixz="0" iyy="1e-6" iyz="0" izz="1e-6" />
                 </inertial>
@@ -466,5 +466,5 @@
               <joint name="joint_lcd_screen" type="fixed">
                 <axis xyz="0 1 0" />
-                <origin xyz=".26 0 0.13" rpy="0 1.57 0"/>
+                <origin xyz=".26 0 0.13" rpy="1.57 0 1.57"/>
                 <parent link="base_link"/>
                 <child link="lcd_screen"/>

Commit message: Update nav
- Add compound map
- Add gmapping launch file
- Update teb planner params

File: mo2bot_description/urdf/mo2bot.xacro (robot description, xacro)
@@ -15,5 +15,5 @@
   <xacro:include filename="$(find mo2bot_description)/urdf/macros.xacro" />
   <!--Moment of Inertia: https://en.wikipedia.org/wiki/List_of_moments_of_inertia, checkout 3D inertial tensor -->
-  <link name='base_link'>
+  <link name="base_link">
     <inertial>
       <mass value="50.0"/>
@@ -26,5 +26,5 @@
         />
       </inertial>
-      <collision name='collision'>
+      <collision name="collision">
         <geometry>
           <box size=".52 .52 .84"/>
@@ -33,5 +33,5 @@
       <!-- The chassis would be split into 2 parts: top & bottom-->
       <!--Top-->
-      <visual name='base_link_visual_top'>
+      <visual name="base_link_visual_top">
         <origin xyz="0 0 0.22" rpy=" 0 0 0"/>
         <geometry>
@@ -40,5 +40,5 @@
       </visual>
       <!--Bottom-->
-      <visual name='base_link_visual_bottom'>
+      <visual name="base_link_visual_bottom">
         <origin xyz="-0.10 0 -0.2" rpy=" 0 0 0"/>
         <geometry>
@@ -47,5 +47,5 @@
       </visual>
       <!--2 beams out-->
-      <visual name='base_link_visual_bottom_left'>
+      <visual name="base_link_visual_bottom_left">
         <origin xyz="0 -0.22 -0.32" rpy=" 0 0 0"/>
         <geometry>
@@ -53,5 +53,5 @@
         </geometry>
       </visual>
-      <visual name='base_link_visual_bottom_right'>
+      <visual name="base_link_visual_bottom_right">
         <origin xyz="0 0.22 -0.32" rpy=" 0 0 0"/>
         <geometry>
@@ -61,6 +61,6 @@
     </link>
     <!--Left trolley wheel-->
-    <link name='trolleyW_wheel_front_left'>
-      <collision name='collision_trolleyW_wheel_front_left'>
+    <link name="trolleyW_wheel_front_left">
+      <collision name="collision_trolleyW_wheel_front_left">
         <origin xyz="0 0 0" rpy=" 0 1.5707 1.5707"/>
         <geometry>
@@ -78,5 +78,5 @@
         </surface>
       </collision>
-      <visual name='visual_trolleyW_wheel_front_left'>
+      <visual name="visual_trolleyW_wheel_front_left">
         <origin xyz="0 0 0" rpy=" 0 1.5707 1.5707"/>
         <geometry>
@@ -102,6 +102,6 @@
       </joint>
       <!--Trolley wheel holder attachment-->
-      <link name='trolleyW_holder_front_left'>
-        <collision name='collision_trolleyW_holder_front_left'>
+      <link name="trolleyW_holder_front_left">
+        <collision name="collision_trolleyW_holder_front_left">
           <origin xyz="-0.03 0 -0.0075" rpy=" 0 0 0"/>
           <geometry>
@@ -119,5 +119,5 @@
           </surface>
         </collision>
-        <visual name='visual_trolleyW_holderHorizontal_front_left'>
+        <visual name="visual_trolleyW_holderHorizontal_front_left">
           <origin xyz="-0.03 0 -0.0075" rpy=" 0 0 0"/>
           <geometry>
@@ -126,5 +126,5 @@
           <material name="grey"/>
         </visual>
-        <visual name='visual_trolleyW_holderVertical_front_left'>
+        <visual name="visual_trolleyW_holderVertical_front_left">
           <origin xyz="-0.04 0 -0.03" rpy=" 0 0 0"/>
           <geometry>
@@ -150,6 +150,6 @@
         </joint>
         <!--Right trolley wheel-->
-        <link name='trolleyW_wheel_front_right'>
-          <collision name='collision_trolleyW_wheel_front_right'>
+        <link name="trolleyW_wheel_front_right">
+          <collision name="collision_trolleyW_wheel_front_right">
             <origin xyz="0 0 0" rpy=" 0 1.5707 1.5707"/>
             <geometry>
@@ -167,5 +167,5 @@
             </surface>
           </collision>
-          <visual name='visual_trolleyW_wheel_front_right'>
+          <visual name="visual_trolleyW_wheel_front_right">
             <origin xyz="0 0 0" rpy=" 0 1.5707 1.5707"/>
             <geometry>
@@ -191,6 +191,6 @@
           </joint>
           <!--Trolley wheel holder attachment-->
-          <link name='trolleyW_holder_front_right'>
-            <collision name='collision_trolleyW_holder_front_right'>
+          <link name="trolleyW_holder_front_right">
+            <collision name="collision_trolleyW_holder_front_right">
               <origin xyz="-0.03 0 -0.0075" rpy=" 0 0 0"/>
               <geometry>
@@ -208,5 +208,5 @@
               </surface>
             </collision>
-            <visual name='visual_trolleyW_holderHorizontal_front_right'>
+            <visual name="visual_trolleyW_holderHorizontal_front_right">
               <origin xyz="-0.03 0 -0.0075" rpy=" 0 0 0"/>
               <geometry>
@@ -215,5 +215,5 @@
               <material name="grey"/>
             </visual>
-            <visual name='visual_trolleyW_holderVertical_front_right'>
+            <visual name="visual_trolleyW_holderVertical_front_right">
               <origin xyz="-0.04 0 -0.03" rpy=" 0 0 0"/>
               <geometry>
@@ -328,5 +328,5 @@
                 </collision>
                 <!--Top-->
-                <visual name='sick_visual_top'>
+                <visual name="sick_visual_top">
                   <origin xyz="0 0 0" rpy="0 0 0"/>
                   <geometry>
@@ -336,5 +336,5 @@
                 </visual>
                 <!--Body-->
-                <visual name='sick_visual_body'>
+                <visual name="sick_visual_body">
                   <origin xyz="0 0 -0.067" rpy="0 0 0"/>
                   <geometry>

Commit message: Add base_footprint link

File: mo2bot_description/urdf/mo2bot.xacro (robot description, xacro)
@@ -16,4 +16,12 @@
   <!--Moment of Inertia: https://en.wikipedia.org/wiki/List_of_moments_of_inertia, checkout 3D inertial tensor -->
   <link name="base_link">
+</link>
+<joint name="baselink_to_basefootprint" type="fixed">
+  <axis xyz="0 0 0"/>
+  <parent link="base_link"/>
+  <child link="base_footprint"/>
+  <origin xyz="0 0 0" rpy="0 0 0" />
+</joint>
+  <link name="base_footprint">
     <inertial>
       <mass value="50.0"/>
